File: stm8s_clock.kicad_pcb (KiCad board)
At the start: 2 copper layers, 157 parts, among them J1 Conn_01x04, J2 PS, Q1 BC847, Q10 BC847, Q11 BC847, Q12 BC847, Q13 BC847, Q14 BC847, Q15 BC847, Q16 BC847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

Commit message: add a new pcb creat
Parts:
- added J3: Conn_01x04, Connector_PinSocket_2.54mm:PinSocket_1x04_P2.54mm_Vertical, F.Cu at (102.5, 150.6)
- added J4: Conn_01x04, Connector_PinSocket_2.54mm:PinSocket_1x04_P2.54mm_Vertical, F.Cu at (107.1, 150.6)
- J2: moved to F.Cu
- moved C7 95.9 mm to (50.6, 87.0), turned to 180 degrees
- moved U4 84.9 mm to (46.7, 90.8), turned to 0 degrees
- moved J1 81.3 mm to (69.0, 100.2), turned to 180 degrees
- moved Y1 80.8 mm to (48.9, 103.1), turned to 0 degrees
- moved BZ1 79.8 mm to (40.0, 126.0), turned to 0 degrees
- moved R1 74.7 mm to (68.8, 95.9), turned to 90 degrees
- moved D1 73.5 mm to (55.1, 108.3), turned to -90 degrees
- moved C2 72.6 mm to (90.8, 104.1), turned to -90 degrees
- moved C5 72.0 mm to (42.5, 103.4)
- moved Q4 70.6 mm to (51.5, 126.1), turned to 180 degrees
- moved C1 69.9 mm to (71.2, 95.9)
- moved C6 66.2 mm to (46.0, 103.4), turned to -90 degrees
- moved R16 63.5 mm to (51.3, 122.3)
- moved C3 56.7 mm to (75.7, 125.7), turned to 90 degrees
- moved C4 56.6 mm to (75.6, 116.1), turned to -90 degrees
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Connections:
- SW1 pad 2: GND -> unconnected-(SW1-Pad2)
- SW2 pad 2: GND -> unconnected-(SW2-Pad2)
- SW3 pad 2: GND -> unconnected-(SW3-Pad2)
- U1 pad 1: unconnected-(U1-PD4-Pad1) -> DAT
- U1 pad 11: unconnected-(U1-PB5-Pad11) -> SW2
- U1 pad 12: unconnected-(U1-PB4-Pad12) -> SW1
- U1 pad 13: unconnected-(U1-PC3-Pad13) -> HT_REST
- U1 pad 14: unconnected-(U1-PC4-Pad14) -> SC
- U1 pad 15: unconnected-(U1-PC5-Pad15) -> SB
- U1 pad 16: unconnected-(U1-PC6-Pad16) -> SA
- U1 pad 17: unconnected-(U1-PC7-Pad17) -> SD
- U1 pad 19: unconnected-(U1-PD2-Pad19) -> HT_CLK
- U1 pad 2: unconnected-(U1-PD5-Pad2) -> LAT
- U1 pad 20: unconnected-(U1-PD3-Pad20) -> HT_IO
- U1 pad 3: unconnected-(U1-PD6-Pad3) -> SCLK
- U1 pad 5: unconnected-(U1-PA1-Pad5) -> SW3
Routing:
- net +12V: track 20.8 -> 199.0 mm, vias 0 -> 6
- net GND: track 89.5 -> 40.0 mm
- net DAT: track 0.00 -> 34.6 mm
- net LAT: track 0.00 -> 31.4 mm
- net SCLK: track 0.00 -> 27.7 mm
- net +5V: track 11.5 -> 33.6 mm
- net Net-(U4-X1): track 11.8 -> 32.3 mm
- net Net-(BT1-+): track 7.20 -> 26.8 mm
- net Net-(J1-Pin_1): track 1.92 -> 18.7 mm
- net Net-(J1-Pin_4): track 0.00 -> 12.9 mm
- net SC: track 0.00 -> 10.3 mm
- net SEL_A: track 163.6 -> 172.6 mm
- net SB: track 0.00 -> 7.53 mm
- net Net-(U1-VCAP): track 3.58 -> 9.59 mm
- net SEL_B: track 258.5 -> 264.0 mm
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Other:
- board outline added: 225.4 x 80 mm
