File: stm8s_clock.kicad_sch (KiCad schematic)
At the start: 158 parts, among them J1 Conn_01x04, J2 PS, Q1 BC847, Q10 BC847, Q11 BC847, Q12 BC847, Q13 BC847, Q14 BC847, Q15 BC847, Q16 BC847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

Commit message: connect to all segment and each digit or shift register to connect each other
Connections:
- net DOT: now also U2.6 (QG)
- net SEGA: now also U2.15 (QA)
- net SEGB: now also U2.2 (QC)
- net SEGC: now also U2.7 (QH)
- net SEGD: now also U2.1 (QB)
- net SEGE: now also U2.5 (QF)
- net SEGF: now also U2.3 (QD)
- net SEGG: now also U2.4 (QE)
Other:
- moved on the sheet: BT1, C5, C6, C7, D1, Q3, Q5, R5, R6, R7, U4, Y1

Commit message: add a new pcb creat
Parts:
- added J3, J4: Conn_01x04, Connector_PinSocket_2.54mm:PinSocket_1x04_P2.54mm_Vertical, symbol Connector_Generic:Conn_01x04
Connections:
- net BUZZER: now also U1.10 (PA3)
- net DAT: now also U1.1 (PD4)
- net GND: now also SW1.3 (K), SW1.4 (A), SW2.3 (K), SW2.4 (A), SW3.3 (K), SW3.4 (A); no longer SW1.2, SW2.2, SW3.2
- net HT_CLK: now also U1.19 (PD2)
- net HT_IO: now also U1.20 (PD3)
- net HT_REST: now also U1.13 (PC3)
- net LAT: now also U1.2 (PD5)
- net SA: now also U1.16 (PC6)
- net SB: now also U1.15 (PC5)
- net SC: now also U1.14 (PC4)
- net SCLK: now also U1.3 (PD6)
- net SD: now also U1.17 (PC7)
- net SW1: now also U1.12 (PB4)
- net SW2: now also U1.11 (PB5)
- net SW3: now also U1.5 (PA1)
